File: Hardware/SparkFun_MMA8452Q-Breakout.sch (EAGLE design)
At the start: 16 parts, among them U1 MMA8452Q

Commit message: removed traces and brand silk for Doug
Parts:
- removed JP1: LOGO-SFESK, SparkFun:LOGO-SFESK
- removed U$1: OSHW-LOGOS, SparkFun:OSHW-LOGOS
Changed lines of the file:
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@@
 <?xml version="1.0" encoding="utf-8"?>
 <!DOCTYPE eagle SYSTEM "eagle.dtd">
-<eagle version="7.3.0">
+<eagle version="7.6.0">
 <drawing>
 <settings>
@@
 <layer number="254" name="cooling" color="7" fill="1" visible="yes" active="yes"/>
 </layers>
-<schematic xreflabel="%F%N/%S" xrefpart="/%S">
+<schematic xreflabel="%F%N/%S" xrefpart="/%S.%C%R">
 <attributes>
 </attributes>
@@
 <part name="P+2" library="SparkFun" deviceset="3.3V" device=""/>
 <part name="P+3" library="SparkFun" deviceset="3.3V" device=""/>
-<part name="U$1" library="SparkFun" deviceset="OSHW-LOGO" device="S"/>
 <part name="U$2" library="SparkFun" deviceset="CREATIVE_COMMONS" device=""/>
-<part name="JP1" library="SparkFun" deviceset="LOGO-SFE" device="SK"/>
 <part name="JP3" library="SparkFun" deviceset="STAND-OFF" device=""/>
 <part name="JP4" library="SparkFun" deviceset="STAND-OFF" device=""/>
@@
 <instance part="P+2" gate="G$1" x="139.7" y="121.92"/>
 <instance part="P+3" gate="G$1" x="147.32" y="121.92"/>
-<instance part="U$1" gate="G$1" x="15.24" y="12.7"/>
 <instance part="U$2" gate="G$1" x="30.48" y="10.16"/>
-<instance part="JP1" gate="G$1" x="241.3" y="17.78"/>
 <instance part="JP3" gate="G$1" x="246.38" y="30.48"/>
 <instance part="JP4" gate="G$1" x="246.38" y="27.94"/>
